File: Apus/Apus.kicad_pcb (KiCad board)
At the start: 2 copper layers, 40 x 24 mm, 18 parts, among them J1 Conn_01x04, J2 Conn_01x04, J3 Conn_01x04_MountingPin, J4 Conn_01x04_MountingPin, U1 TMAG5273A2QDBVR

Commit message: feat: add Qwiic connector (symbol + footprint + PCB placement)
Parts:
- added G***: LOGO, SparkFun-Qwiic:qwiic_3mm, F.Cu at (202.0, 74.0)
- moved C1 8.95 mm to (221.0, 72.7)
- moved D1 8.95 mm to (206.2, 74.0)
- moved H1 8.95 mm to (202.7, 62.0)
- moved H2 8.95 mm to (234.7, 62.0)
- moved H3 8.95 mm to (202.7, 78.0)
- moved H4 8.95 mm to (234.7, 78.0)
- moved J1 8.95 mm to (214.9, 80.2)
- moved J2 8.95 mm to (214.9, 59.8)
- moved J3 8.95 mm to (202.0, 70.0)
- moved J4 8.95 mm to (235.4, 70.0)
- moved JP2 8.95 mm to (217.7, 72.4)
- moved JP3 8.95 mm to (206.1, 71.2)
- moved R2 8.95 mm to (216.9, 66.0)
- moved R3 8.95 mm to (221.1, 66.0)
- moved U1 8.95 mm to (219.0, 70.0)
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