File: Apus/Apus.kicad_sch (KiCad schematic)
At the start: 0 parts

Commit message: feat: initial schematic for TMAG5273 Qwiic module
- Add TMAG5273 3D Hall-effect sensor
- Add Qwiic connectors and breadboard header
- Add I2C pull-ups, LED indicator, and decoupling
- Set title block to v1.0.0
Parts:
- added C1: 100nF, Capacitor_SMD:C_0603_1608Metric, symbol Device:C
- added D1: LED, LED_SMD:LED_0603_1608Metric, symbol Device:LED
- added H1, H2, H3, H4: MountingHole, MountingHole:MountingHole_3.2mm_M3, symbol Mechanical:MountingHole
- added J1: Conn_01x04, Connector_PinHeader_2.54mm:PinHeader_1x04_P2.54mm_Vertical, symbol Connector_Generic:Conn_01x04
- added J2, J3: Conn_01x04_MountingPin, Connector_JST:JST_SH_SM04B-SRSS-TB_1x04-1MP_P1.00mm_Horizontal, symbol Connector_Generic_MountingPin:Conn_01x04_MountingPin
- added JP1: SolderJumper_3_Bridged123, Jumper:SolderJumper-3_P1.3mm_Bridged12_RoundedPad1.0x1.5mm_NumberLabels, symbol Jumper:SolderJumper_3_Bridged123
- added JP2, JP3: SolderJumper_2_Bridged, Jumper:SolderJumper-2_P1.3mm_Bridged_RoundedPad1.0x1.5mm, symbol Jumper:SolderJumper_2_Bridged
- added R1: 4.7k, Resistor_SMD:R_0603_1608Metric, symbol Device:R
- added R2, R3: 2.2k, Resistor_SMD:R_0603_1608Metric, symbol Device:R
- added R4: 10k, Resistor_SMD:R_0603_1608Metric, symbol Device:R
- added U1: TMAG5273A2QDBVR, TMAG5273A2QDBVR:SOT95P280X140-6N, symbol TMAG5273A2QDBVR:TMAG5273A2QDBVR
Connections:
- new net: JP1.1 (A), R3.1
- new net: JP1.3 (B), R2.1
- new net: D1.1 (K), JP3.2 (B)
- new net: JP2.1 (A), R4.1
- new net: D1.2 (A), R1.2
- new net +3V3: C1.1, J1.1 (Pin_1), J2.2 (Pin_2), J3.2 (Pin_2), JP1.2 (C), JP2.2 (B), R1.1, U1.4 (VCC)
- new net GND: C1.2, J1.2 (Pin_2), J2.1 (Pin_1), J2.MP (MountPin), J3.1 (Pin_1), J3.MP (MountPin), JP3.1 (A), U1.2 (GND), U1.3 (TEST)
- new net SCL: J1.4 (Pin_4), J2.4 (Pin_4), J3.4 (Pin_4), R2.2, U1.1 (SCL)
- new net SDA: J1.3 (Pin_3), J2.3 (Pin_3), J3.3 (Pin_3), R3.2, U1.6 (SDA)
- new net ~{INT}: R4.2, U1.5 (~{INT})
Other:
- company: (none) -> Vion Qaro
- title: (none) -> Apus

Commit message: feat: initial PCB release v1.0.0
- Final PCB layout (Gerber, drill, pick-and-place)
- Complete BOM with MPN
- Production folder ready for fab house
- Schematic, stack-up, and DRC report

Note:
- Not physically tested (engineering sample)
- Not ready for mass production
Parts:
- removed H1, H2, H3, H4: MountingHole, MountingHole:MountingHole_3.2mm_M3, symbol Mechanical:MountingHole
- added H1, H2, H3, H4: MountingHole_Pad, MountingHole:MountingHole_3.2mm_M3_Pad, symbol Mechanical:MountingHole_Pad
- added J2: Conn_01x04, Connector_PinHeader_2.54mm:PinHeader_1x04_P2.54mm_Vertical, symbol Connector_Generic:Conn_01x04
- JP1: footprint Jumper:SolderJumper-3_P1.3mm_Bridged12_RoundedPad1.0x1.5mm_NumberLabels -> Jumper:SolderJumper-3_P1.3mm_Bridged123_RoundedPad1.0x1.5mm_NumberLabels
- renumbered J2 to J3, J3 to J4
Connections:
- net +3V3: now also J1.2 (Pin_2), J2.2 (Pin_2); no longer J1.1 (Pin_1)
- net GND: now also J1.1 (Pin_1), J1.4 (Pin_4), H1.1, H2.1, H3.1, H4.1, J2.1 (Pin_1); no longer J1.2 (Pin_2)
- net SCL: now also J2.4 (Pin_4); no longer J1.4 (Pin_4)
- net SDA: now also J2.3 (Pin_3); no longer J1.3 (Pin_3)
- net ~{INT}: now also J1.3 (Pin_3)

Commit message: feat: add Qwiic connector (symbol + footprint + PCB placement)
Parts:
- added G1: qwiic_Logo, Package_QFP:TQFP-44_10x10mm_P0.8mm, symbol SparkFun-Qwiic:qwiic_Logo
Changed lines of the file:
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@@
+	)
+	(symbol
+		(lib_id "SparkFun-Qwiic:qwiic_Logo")
+		(at 113.03 130.81 0)
+		(unit 1)
+		(body_style 1)
+		(exclude_from_sim no)
+		(in_bom yes)
+		(on_board no)
+		(in_pos_files yes)
+		(dnp no)
+		(fields_autoplaced yes)
+		(property "Reference" "G1"
+			(at 113.03 127 0)
+			(hide yes)
+			(show_name no)
+			(do_not_autoplace no)
+			(effects
+				(font
+					(size 1.27 1.27)
+				)
+			)
+		)
+		(property "Value" "qwiic_Logo"
+			(at 113.03 134.62 0)
+			(hide yes)
+			(show_name no)
+			(do_not_autoplace no)
+			(effects
+				(font
+					(size 1.27 1.27)
+				)
+			)
+		)
+		(property "Footprint" "Package_QFP:TQFP-44_10x10mm_P0.8mm"
+			(at 113.03 137.16 0)
+			(hide yes)
+			(show_name no)
+			(do_not_autoplace no)
+			(effects
+				(font
+					(size 1.27 1.27)
+				)
+			)
+		)
+		(property "Datasheet" ""
+			(at 113.03 130.81 0)
+			(hide yes)
+			(show_name no)
+			(do_not_autoplace no)
+			(effects
+				(font
+					(size 1.27 1.27)
+				)
+			)
+		)
+		(property "Description" ""
+			(at 113.03 130.81 0)
+			(hide yes)
+			(show_name no)
+			(do_not_autoplace no)
+			(effects
+				(font
+					(size 1.27 1.27)
+				)
+			)
+		)
+		(instances
+			(project "Apus"
+				(path "/5099b96d-ff89-41f5-8045-2c8201a79f0f"
+					(reference "G1")
+					(unit 1)
+				)
+			)
+		)
 	)
 	(symbol
